File: Proyecto RoomLink/RoomLink/Control.kicad_sch (KiCad schematic)
At the start: 31 parts, among them IC1 MKE04Z128VLD4, J2 Jtag_Conector_PdX, SW1 SW_MEC_5E, Y1 8Mhz

Commit message: Update
Parts:
- removed C1 (x2): 22pF/50V, Capacitor_SMD:C_0805_2012Metric, symbol pdxlbs:C_small_.1uf_PDX
- removed C1: 0.1uF/50V, Capacitor_SMD:C_0805_2012Metric, symbol pdxlbs:C_small_.1uf_PDX
- removed D19: LED_Small_Filled, LED_SMD:LED_0805_2012Metric_Pad1.15x1.40mm_HandSolder, symbol Device:LED_Small_Filled
- removed IC1: MKE04Z128VLD4, QFP80P1200X1200X160-44N, symbol MKE04Z128VLD4:MKE04Z128VLD4
- removed J2: Jtag_Conector_PdX, w_smd_plcc:Jtag_PdX_TAG_TC2030-IDC-NL, symbol pdxlbs:Jtag_Conector_PdX
- removed J5: ~, symbol MCE_LIB:JTAG_SWD
- removed R34: 470, Resistor_SMD:R_0805_2012Metric_Pad1.20x1.40mm_HandSolder, symbol Device:R_Small
- removed R35, R36, R37, R38, R39, R40, R41, R42, R43, R45, R46, R47, R48: 10k, Resistor_SMD:R_0805_2012Metric_Pad1.20x1.40mm_HandSolder, symbol Device:R_Small
- removed R44: 10M, Resistor_SMD:R_0805_2012Metric_Pad1.20x1.40mm_HandSolder, symbol Device:R_Small
- removed R49: 100k, Resistor_SMD:R_0805_2012Metric_Pad1.20x1.40mm_HandSolder, symbol Device:R_Small
- removed R50, R51: 100K, Resistor_SMD:R_0805_2012Metric_Pad1.20x1.40mm_HandSolder, symbol Device:R_Small
- removed R52, R53: 1K, Resistor_SMD:R_0805_2012Metric_Pad1.20x1.40mm_HandSolder, symbol Device:R_Small
- removed S1: ~, symbol MCE_LIB:Dip_Switch_08
- removed S2: ~, symbol MCE_LIB:Dip_Switch_04
- removed SW1: SW_MEC_5E, symbol Switch:SW_MEC_5E
- removed Y1: 8Mhz, symbol Device:Crystal_Small
- added C1: 22uF, Capacitor_SMD:C_0805_2012Metric, symbol componets_new:C
- added C2, C3: 0.1uF, Capacitor_SMD:C_0805_2012Metric, symbol componets_new:C
- added D1: LED, LED_SMD:LED_0805_2012Metric, symbol Device:LED
- added J3: Conn_ARM_JTAG_SWD_10, Connector_PinHeader_1.27mm:PinHeader_2x05_P1.27mm_Vertical, symbol Connector:Conn_ARM_JTAG_SWD_10
- added R1: 470, Resistor_SMD:R_0805_2012Metric, symbol Device:R
- added R2: 22K, Resistor_SMD:R_0805_2012Metric, symbol Device:R
- added R3, R4, R5, R6, R7: 1K, Resistor_SMD:R_0805_2012Metric, symbol Device:R
- added U1: ESP32-WROOM-32, LibKiCad:ESP32WROOM32EN4, symbol RF_Module:ESP32-WROOM-32
- added U2: ~, LibKiCad:PinHeader2x3, symbol componets_new:PinHeader
Connections:
- net COM_RS485_LCD: now also U1.6 (IO34)
- net CON_RS485_eXT: now also U1.7 (IO35)
- net GND: now also C1.2, C2.2, D1.1 (K), J3.3 (GND), J3.5 (GND), U1.1 (GND), U1.15 (GND), U1.38 (GND), U1.39 (GND), U2.5
- net INPUT_1_MICRO: now also U1.25 (IO0)
- net INPUT_2_MICRO: now also U1.29 (IO5)
- net INPUT_3_MICRO: now also U1.26 (IO4)
- net INPUT_4_MICRO: now also U1.24 (IO2)
- net RLY_FAN1_MICRO: now also U1.10 (IO25)
- net RLY_FAN2_MICRO: now also U1.11 (IO26)
- net RLY_FAN3_MICRO: now also U1.12 (IO27)
- net RLY_OUT1_MICRO: now also U1.36 (IO22)
- net RLY_OUT2_MICRO: now also U1.37 (IO23)
- net Rx_RS485_LCD: now also U1.27 (IO16)
- net Rx_RS485_eXT: now also U1.34 (RXD0/IO3)
- net Tx_RS485_LCD: now also U1.28 (IO17)
- net Tx_RS485_eXT: now also U1.35 (TXD0/IO1)
- new net: D1.2 (A), R1.2
- new net: U1.30 (IO18), U2.2
- new net: U1.31 (IO19), U2.4
- new net: U1.33 (IO21), U2.6
- new net: J3.1 (VTref), R3.2
- new net +3.3V: C1.1, C2.1, C3.1, R2.1, R3.1, R4.1, R5.1, R6.1, R7.1, U1.2 (VDD), U2.1
- new net IO32: U1.8 (IO32), U2.3
- new net IO33: R1.1, U1.9 (IO33)
- new net SWCLK: J3.4 (SWDCLK/TCK), R5.2, U1.16 (IO13)
- new net SWDIO: J3.2 (SWDIO/TMS), R6.2, U1.13 (IO14)
- new net SWO: J3.6 (SWO/TDO), U1.23 (IO15)
- new net TDI: J3.8 (NC/TDI), R7.2, U1.14 (IO12)
- new net ~Reset: C3.2, J3.10 (~{RESET}), R2.2, R4.2, U1.3 (EN)
- no-connect marks 0 -> 9
