File: Proyecto RoomLink/RoomLink/INPUTS.kicad_sch (KiCad schematic)
At the start: 28 parts, among them U1 FODM2705

Commit message: Update
Parts:
- renumbered C3 to C10, C2 to C11, C4 to C12, C1 to C9, D1 to D?, R1 to R?, U1 to U?
Connections:
- net +12V is gone; now on net VDD: R?.2, R?.2, R?.2, R?.2, R?.2, R?.2, R?.2, R?.2
- net VDD: no longer R?.2, R?.2, R?.2, R?.2
- new net +3.3V: R?.2, R?.2, R?.2, R?.2
Other:
- moved on the sheet: D?, R?
