File: Proyecto RoomLink/RoomLink/RELAY_GROUP.kicad_sch (KiCad schematic)
At the start: 16 parts, among them K1 AZ921, U1 ULN2003

Commit message: Update
Parts:
- renumbered D1 to D?, K1 to K?, R1 to R?, U1 to U?
