File: Proyecto RoomLink/RoomLink/RS-485_Externa.kicad_sch (KiCad schematic)
At the start: 11 parts

Commit message: Update
Parts:
- F2: renamed from F1; footprint (none) -> LibKiCad:PTS120660V010
- F3: renamed from F2; footprint (none) -> LibKiCad:PTS120660V010
- renumbered D11 to D18, D12 to D19, D1 to D?, PS1 to PS2, R1 to R?
