File: Proyecto RoomLink/RoomLink/RS-485_LCD.kicad_sch (KiCad schematic)
At the start: 8 parts, among them U6 SP485ECN-L/TR

Commit message: Update
Parts:
- renumbered C1 to C?, D11 to D?, D12 to D?, R1 to R?, U6 to U3
Connections:
- net +5V renamed +12V
Other:
- moved on the sheet: C?
