File: Proyecto RoomLink/RoomLink/RoomLink.kicad_sch (KiCad schematic)
At the start: 6 parts, among them J1 TBP03R1-350-02BE, J4 TBP03R1-350-02BE

Commit message: Update
Parts:
- renumbered ENTRADA_AC to ENTRADA_AC1, ENTRADA_RS485 to ENTRADA_RS1, INPUT to INPUT1, J4 to J2, OUTPUT to OUTPUT1
Changed lines of the file:
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@@
   (symbol (lib_id "TBP03R1-350-08BE:TBP03R1-350-08BE") (at 112.522 114.808 0) (mirror y) (unit 1)
     (in_bom yes) (on_board yes) (dnp no)
-    (property "Reference" "INPUT" (at 105.664 112.268 0)
+    (property "Reference" "INPUT1" (at 105.664 112.268 0)
       (effects (font (size 1.27 1.27)) (justify left))
     )
@@
       (project "RoomLink"
         (path "/a574160c-788b-41d3-8a5c-f7edad3dde0f"
-          (reference "INPUT") (unit 1)
+          (reference "INPUT1") (unit 1)
         )
       )
@@
   (symbol (lib_id "TBP03R1-350-03BE:TBP03R1-350-03BE") (at 112.268 89.916 0) (mirror y) (unit 1)
     (in_bom yes) (on_board yes) (dnp no)
-    (property "Reference" "ENTRADA_RS485" (at 105.41 88.646 0)
+    (property "Reference" "ENTRADA_RS1" (at 105.41 88.646 0)
       (effects (font (size 1.27 1.27)) (justify left))
     )
@@
       (project "RoomLink"
         (path "/a574160c-788b-41d3-8a5c-f7edad3dde0f"
-          (reference "ENTRADA_RS485") (unit 1)
+          (reference "ENTRADA_RS1") (unit 1)
         )
       )
@@
   (symbol (lib_id "TBP03R1-350-08BE:TBP03R1-350-08BE") (at 188.214 114.808 0) (unit 1)
     (in_bom yes) (on_board yes) (dnp no) (fields_autoplaced)
-    (property "Reference" "OUTPUT" (at 194.818 113.538 0)
+    (property "Reference" "OUTPUT1" (at 194.818 113.538 0)
       (effects (font (size 1.27 1.27)) (justify left))
     )
@@
       (project "RoomLink"
         (path "/a574160c-788b-41d3-8a5c-f7edad3dde0f"
-          (reference "OUTPUT") (unit 1)
+          (reference "OUTPUT1") (unit 1)
         )
       )
@@
   (symbol (lib_id "TBP03R1-350-02BE:TBP03R1-350-02BE") (at 112.268 76.962 0) (mirror y) (unit 1)
     (in_bom yes) (on_board yes) (dnp no)
-    (property "Reference" "ENTRADA_AC" (at 106.172 74.422 0)
+    (property "Reference" "ENTRADA_AC1" (at 106.172 74.422 0)
       (effects (font (size 1.27 1.27)) (justify left))
     )
@@
       (project "RoomLink"
         (path "/a574160c-788b-41d3-8a5c-f7edad3dde0f"
-          (reference "ENTRADA_AC") (unit 1)
+          (reference "ENTRADA_AC1") (unit 1)
         )
       )
@@
   (symbol (lib_id "TBP03R1-350-02BE:TBP03R1-350-02BE") (at 188.214 89.916 0) (unit 1)
     (in_bom yes) (on_board yes) (dnp no) (fields_autoplaced)
-    (property "Reference" "J4" (at 194.31 87.376 0)
+    (property "Reference" "J2" (at 194.31 87.376 0)
       (effects (font (size 1.27 1.27)) (justify left))
     )
@@
       (project "RoomLink"
         (path "/a574160c-788b-41d3-8a5c-f7edad3dde0f"
-          (reference "J4") (unit 1)
+          (reference "J2") (unit 1)
         )
       )
