File: Proyecto RoomLink/RoomLink/Power_supply.kicad_sch.kicad_sch (KiCad schematic)
At the start: 20 parts, among them U7 7805

Commit message: Update
Parts:
- removed F4, F5: Fuse, symbol Device:Fuse
- removed PS3: B0505S-2WR2, LibKiCad:B0505S2WR2, symbol B0505S-2WR2:B0505S-2WR2
- removed U7: 7805, symbol pdxlbs:7805
- removed Z2: 1SMA5919BT3G, LibKiCad:DIONM5436X261N, symbol 1SMA5919BT3G:1SMA5919BT3G
- added U5: LM1117MP-3.3, Package_TO_SOT_SMD:SOT-223-3_TabPin2, symbol Regulator_Linear:LM1117MP-3.3
- C8: renamed from C9; footprint (none) -> Capacitor_SMD:CP_Elec_5x5.4
- F1: renamed from F3; footprint (none) -> LibKiCad:fuse20x5
- R?: renamed from R1; value 1K -> 470
- R?: renamed from R1; value 1K -> 2.2K
- TVS1: footprint (none) -> Varistor:RV_Disc_D12mm_W6.7mm_P7.5mm
- renumbered C1 to C?, D1 to D?, PS2 to PS1, R1 to R?
Connections:
- net CON_DC+ is gone; now on net +12V: R?.2
- net CON_DC- is gone; now on net Earth: D?.1 (K)
- net +12V: now also U5.3 (VI)
- net CON_L1: now also PS1.1 (AC/L), TVS1.2; no longer F1.1
- net CON_NEUT: now also F1.1; no longer PS1.1 (AC/L), TVS1.1
- net Earth: now also U5.1 (GND)
- net at F1.2, PS1.2 (AC/N): now also TVS1.1; no longer TVS1.2
- net +5V renamed +3.3V
- net +3.3V: now also U5.2 (VO)
Other:
- moved on the sheet: C8, C?, D?, F1, R?, Z1

Commit message: Up
Parts:
- added U10: B_S-2WR2, LibKiCad:B_S-2WR2, symbol componets_new:B_S-2WR2
- added Z2: 1SMA5919BT3G, LibKiCad:DIONM5436X261N, symbol 1SMA5919BT3G:1SMA5919BT3G
Connections:
- net +3.3V: now also U10.4 (Vo), Z2.1 (K); no longer C8.1, C?.1, U5.2 (VO), Z1.1 (K)
- net Earth: now also U10.3 (0V), Z2.2 (A)
- net GND: now also U10.1 (GND)
- net VDD: now also C8.1, C?.1, U5.2 (VO), Z1.1 (K), U10.2 (Vin)
Other:
- moved on the sheet: D?, R?
