File: Proyecto RoomLink/RoomLink/RoomLink.kicad_pcb (KiCad board)
At the start: 2 copper layers, 102.4 x 83.1 mm, 99 parts, among them J1 TBP03R1-350-02BE, J2 TBP03R1-350-02BE, J3 Conn_ARM_JTAG_SWD_10, K1 AZ921, K2 AZ921, K3 AZ921, K4 AZ921, K5 AZ921, U1 ESP32-WROOM-32, U3 SP485ECN-L/TR, U4 ULN2003, U5 LM1117MP-3.3, U6 FODM2705, U7 FODM2705, U8 FODM2705, U9 FODM2705

Commit message: Up
Parts:
- added U10: B_S-2WR2, LibKiCad:B_S-2WR2, F.Cu at (153.9, 97.3)
- added Z2: 1SMA5919BT3G, LibKiCad:DIONM5436X261N, F.Cu at (150.5, 106.3)
- moved C12 155.0 mm to (228.6, 145.0)
- moved D16 155.0 mm to (228.8, 132.9)
- moved R23 155.0 mm to (205.0, 132.6)
- moved R25 155.0 mm to (205.0, 138.5)
- moved R31 155.0 mm to (209.7, 138.5)
- moved R35 155.0 mm to (214.5, 132.6)
- moved C10 155.0 mm to (228.6, 138.9)
- moved D14 155.0 mm to (228.8, 126.8)
- moved R27 155.0 mm to (209.7, 126.7)
- moved R32 155.0 mm to (214.5, 123.7)
- moved R20 146.2 mm to (194.3, 129.8), turned to -90 degrees
- moved R22 137.3 mm to (186.7, 129.8), turned to 90 degrees
- moved R24 135.7 mm to (188.0, 121.9), turned to 180 degrees
- moved R26 130.5 mm to (186.3, 116.2)
- moved R28 130.2 mm to (184.2, 129.8), turned to -90 degrees
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Connections:
- C7 pad 1: +3.3V -> VDD
- C8 pad 1: +3.3V -> VDD
- U5 pad 2: +3.3V -> VDD
- Z1 pad 1: +3.3V -> VDD
